Commit message: Added tutorial_data_collection.py and solution

File: robotac_sim/descriptions/camera/azure.urdf (robot description, URDF)
Before this commit: robot azure-kinect, 3 links, 2 joints
Links:
- added link camera_baselink, mass 1.0
- link camera_base: mass None -> 1.0
- link camera_body: mass None -> 1.0
- link camera_visor: mass None -> 1.0
Joints:
- added joint camera_baselink_to_base: type fixed, parent camera_baselink, child camera_base, origin xyz=0 0. 0 rpy=0. 1.57 1.57
