Commit message: Updated tutorial files

File: robotac_sim/descriptions/ycb_objects/YcbChipsCan_1/model.urdf (robot description, URDF)
Before this commit: robot model.urdf, 1 links, 0 joints
Links:
- link baseLink: mass 0.15 -> 0.175

File: robotac_sim/descriptions/ycb_objects/YcbHammer_1/model.urdf (robot description, URDF)
Before this commit: robot model.urdf, 1 links, 0 joints
Links:
- link baseLink: mass .2 -> .1; geometry collision mesh filename=collision_vhacd.obj scale=1 1.2 1.2; visual mesh filename=textured_reoriented.obj scale=1 1.2 1.2
