Commit message: Updated solution files for large datacollection

File: robotac_sim/descriptions/ycb_objects/YcbBanana_2/model.urdf (robot description, URDF)
Before this commit: robot model.urdf, 1 links, 0 joints
Links:
- link baseLink: mass .066 -> .1

File: robotac_sim/descriptions/ycb_objects/YcbHammer_2/model.urdf (robot description, URDF)
Before this commit: robot model.urdf, 1 links, 0 joints
Links:
- link baseLink: mass .2 -> .125

File: robotac_sim/descriptions/ycb_objects/YcbHammer_3/model.urdf (robot description, URDF)
Before this commit: robot model.urdf, 1 links, 0 joints
Links:
- link baseLink: mass .2 -> .1

File: robotac_sim/descriptions/ycb_objects/YcbMustardBottle_2/model.urdf (robot description, URDF)
Before this commit: robot model.urdf, 1 links, 0 joints
Links:
- link baseLink: mass .105 -> .125
